Commit message: copied own racer description for gazebo due problems with position and rotation

File: ros_ws/src/simulation/racer_description/urdf/racer-kinect.xacro (robot description, xacro)
@@ -78,6 +78,5 @@
     </collision>
     <visual>
-	    <!--<origin xyz="0 0.08 0.09" rpy="0 -1.570796327 -1.570796327"/>-->
-      <origin xyz="0 0 0" rpy="0 0 0"/>
+      <origin xyz="0 0.08 0.09" rpy="0 -1.570796327 -1.570796327"/>
       <geometry>
         <mesh filename="package://racer_description/meshes/ZED.dae"/>
