Commit message: added depth camera

File: ros_ws/src/simulation/racer_description/urdf/racer.xacro (robot description, xacro)
@@ -83,5 +83,5 @@
       </geometry>
     </visual>
-  </link>s
+  </link>
   <joint name="camera_joint" type="fixed">
     <axis xyz="0 1 0" />

Commit message: depth cam now included with correct orientation

File: ros_ws/src/simulation/racer_description/urdf/racer.xacro (robot description, xacro)
@@ -78,5 +78,5 @@
     </collision>
     <visual>
-      <origin xyz="0 0 0" rpy="0 0 0"/>
+      <origin xyz="0 0.08 0.09" rpy="0 -1.570796327 -1.570796327"/>
       <geometry>
         <mesh filename="package://racer_description/meshes/ZED.dae"/>

Commit message: moved lidar to correct position in simulation model

File: ros_ws/src/simulation/racer_description/urdf/racer.xacro (robot description, xacro)
@@ -104,5 +104,6 @@
     </collision>
     <visual>
-      <origin xyz="0 0 ${wheel_height/2}" rpy="0 0 0"/>
+      <!--<origin xyz="0 0 ${wheel_height/2}" rpy="0 0 0"/>-->
+      <origin xyz="0 0 -0.02" rpy="0 0 0"/>
       <geometry>
         <mesh filename="package://racer_description/meshes/hokuyo.dae"/>

Commit message: aligned camera in visualization

File: ros_ws/src/simulation/racer_description/urdf/racer.xacro (robot description, xacro)
@@ -78,6 +78,5 @@
     </collision>
     <visual>
-	    <!--<origin xyz="0 0.08 0.09" rpy="0 -1.570796327 -1.570796327"/>-->
-      <origin xyz="0 0 0" rpy="0 0 0"/>
+      <origin xyz="0.060 0 -0.08" rpy="0 0 0"/>
       <geometry>
         <mesh filename="package://racer_description/meshes/ZED.dae"/>

Commit message: final camera adjustments, solves #13

File: ros_ws/src/simulation/racer_description/urdf/racer.xacro (robot description, xacro)
@@ -78,5 +78,5 @@
     </collision>
     <visual>
-      <origin xyz="0.060 0 -0.08" rpy="0 0 0"/>
+      <origin xyz="0.260 0 -0.0125" rpy="0 0 0"/>
       <geometry>
         <mesh filename="package://racer_description/meshes/ZED.dae"/>
@@ -86,5 +86,5 @@
   <joint name="camera_joint" type="fixed">
     <axis xyz="0 1 0" />
-    <origin xyz="0.21 0 0.095" rpy="0 0 0"/>
+    <origin xyz="0.01 0 0.0" rpy="0 0 0"/>
     <parent link="chassis"/>
     <child link="camera"/>
